File: PCB macropad/macro pad.kicad_pcb (KiCad board)
At the start: 2 copper layers, 69.9 x 69.9 mm, 12 parts, among them SW1 SW_Push, SW2 SW_Push, SW3 SW_Push, SW4 SW_Push, SW5 RotaryEncoder_Switch, U1 MOUDLE-SEEEDUINO-XIAO, U2 ER_OLEDM0.91_1x-I2C

Commit message: Update all project files
Parts:
- moved U1 7.46 mm to (162.5, 120.0)
- moved SW4 5.08 mm to (184.9, 97.5)
- moved SW1 5.00 mm to (184.9, 77.5)
- moved SW2 5.00 mm to (184.9, 117.5)
- moved SW3 5.00 mm to (164.9, 97.5)
- moved SW5 5.00 mm to (167.5, 87.2)
Routing:
- net /SDA: track 44.3 -> 26.2 mm, vias 2 -> 0
- net Net-(U1-PB08_A6_D6_TX): track 73.3 -> 57.6 mm, vias 5 -> 2
- net /SCL: track 35.1 -> 49.4 mm, vias 2 -> 0
- net GND: track 127.1 -> 113.3 mm, vias 5 -> 3
- net Net-(U1-PB09_A7_D7_RX): track 33.6 -> 20.9 mm
- net Net-(U1-PA5_A9_D9_MISO): track 36.3 -> 23.8 mm
- net Net-(U1-PA10_A2_D2): track 52.9 -> 62.4 mm, vias 5 -> 2
- net /VCC: track 10.3 -> 4.70 mm
- net Net-(U1-PA6_A10_D10_MOSI): track 51.2 -> 46.6 mm, vias 0 -> 3
- net Net-(U1-PA11_A3_D3): track 58.9 -> 56.4 mm, vias 1 -> 2
- net Net-(U1-PA7_A8_D8_SCK): track 19.0 -> 17.6 mm

Commit message: Update all project files
Parts:
- moved U1 2.54 mm to (165.0, 120.0), turned to 180 degrees
- moved REF** 1.00 mm to (206.0, 130.0)
- moved REF** 1.00 mm to (206.0, 70.0)
Routing:
- net GND: track 113.3 -> 144.9 mm, vias 3 -> 5
- net /SCL: track 49.4 -> 27.0 mm, vias 0 -> 2
- net /VCC: track 4.70 -> 26.4 mm
- net Net-(U1-PA11_A3_D3): track 56.4 -> 37.8 mm
- net Net-(U1-PA10_A2_D2): track 62.4 -> 45.5 mm
- net Net-(U1-PB08_A6_D6_TX): track 57.6 -> 40.9 mm
- net Net-(U1-PA5_A9_D9_MISO): track 23.8 -> 38.2 mm
- net Net-(U1-PB09_A7_D7_RX): track 20.9 -> 34.5 mm, vias 0 -> 4
- net Net-(U1-PA6_A10_D10_MOSI): track 46.6 -> 57.7 mm, vias 3 -> 4
- net Net-(U1-PA7_A8_D8_SCK): track 17.6 -> 20.7 mm
- net /SDA: track 26.2 -> 28.0 mm, vias 0 -> 2
